Commit message: Issue happening with joint_limits.yaml no accel

File: install/ur3e_gazebo_sim/share/ur3e_gazebo_sim/urdf/ur3e_common.xacro (robot description, xacro)
@@ -15,24 +15,30 @@
     <xacro:property name="shoulder_pan_velocity_limit" value="3.1416" scope="parent"/>
     <xacro:property name="shoulder_pan_effort_limit" value="56.0" scope="parent"/>
+    <xacro:property name="shoulder_pan_accel_limit" value = "3.1416" scope="parent"/>
     <xacro:property name="shoulder_lift_lower_limit" value="-6.2832" scope="parent"/>
     <xacro:property name="shoulder_lift_upper_limit" value="6.2832" scope="parent"/>
     <xacro:property name="shoulder_lift_velocity_limit" value="3.1416" scope="parent"/>
     <xacro:property name="shoulder_lift_effort_limit" value="56.0" scope="parent"/>
+    <xacro:property name="shoulder_lift_accel_limit" value = "3.1416" scope="parent"/>
     <xacro:property name="elbow_joint_lower_limit" value="-3.1416" scope="parent"/>
     <xacro:property name="elbow_joint_upper_limit" value="3.1416" scope="parent"/>
     <xacro:property name="elbow_joint_velocity_limit" value="3.1416" scope="parent"/>
     <xacro:property name="elbow_joint_effort_limit" value="28.0" scope="parent"/>
+    <xacro:property name="elbot_joint_accel_limit" value = "3.1416" scope="parent"/>
     <xacro:property name="wrist_1_lower_limit" value="-6.2832" scope="parent"/>
     <xacro:property name="wrist_1_upper_limit" value="6.2832" scope="parent"/>
     <xacro:property name="wrist_1_velocity_limit" value="6.2832" scope="parent"/>
     <xacro:property name="wrist_1_effort_limit" value="12.0" scope="parent"/>
+    <xacro:property name="wrist_1_accel_limit" value = "3.1416" scope="parent"/>
     <xacro:property name="wrist_2_lower_limit" value="-6.2832" scope="parent"/>
     <xacro:property name="wrist_2_upper_limit" value="6.2832" scope="parent"/>
     <xacro:property name="wrist_2_velocity_limit" value="6.2832" scope="parent"/>
     <xacro:property name="wrist_2_effort_limit" value="12.0" scope="parent"/>
+    <xacro:property name="wrist_2_accel_limit" value = "3.1416" scope="parent"/>
     <xacro:property name="wrist_3_lower_limit" value="-6.2832" scope="parent"/>
     <xacro:property name="wrist_3_upper_limit" value="6.2832" scope="parent"/>
     <xacro:property name="wrist_3_velocity_limit" value="6.2832" scope="parent"/>
     <xacro:property name="wrist_3_effort_limit" value="12.0" scope="parent"/>
+    <xacro:property name="wrist_3_accel_limit" value = "3.1416" scope="parent"/>
     <xacro:property name="d1" value="0.1519" scope="parent"/>
     <xacro:property name="a2" value="-0.24365" scope="parent"/>

File: install/ur3e_gazebo_sim/share/ur3e_gazebo_sim/urdf/ur3e_macro.urdf.xacro (robot description, xacro)
@@ -160,7 +160,5 @@
             <axis xyz="0.0 0.0 1.0"/>
             <limit lower="${shoulder_pan_lower_limit}" upper="${shoulder_pan_upper_limit}" effort="${shoulder_pan_effort_limit}" velocity="${shoulder_pan_velocity_limit}"/>
-            <xacro:if value="${safety_limits}">
-                <safety_controller soft_lower_limit="${shoulder_pan_lower_limit + safety_pos_margin}" soft_upper_limit="${shoulder_pan_upper_limit - safety_pos_margin}" k_position="${safety_k_position}" k_velocity="0.0"/>
-            </xacro:if>
+            <safety_controller soft_lower_limit="${shoulder_pan_lower_limit + safety_pos_margin}" soft_upper_limit="${shoulder_pan_upper_limit - safety_pos_margin}" k_position="${safety_k_position}" k_velocity="0.0"/>
             <dynamics damping="0" friction="1"/>
         </joint>

File: install/ur3e_gazebo_sim/share/ur3e_gazebo_sim/urdf/ur3e_ros2_control.xacro (robot description, xacro)
@@ -6,4 +6,5 @@
             <gazebo>
                 <plugin filename="libgazebo_ros2_control.so" name="gazebo_ros2_control">
+                    <robot_sim_type>gazebo_ros2_control/GazeboSystem</robot_sim_type>
                     <parameters>$(find ur3e_gazebo_sim)/config/ur3e_controller.yaml</parameters>
                 </plugin>
@@ -27,5 +28,5 @@
                 <state_interface name="effort"/>
             </joint>
-            <joint name="${prefix}shoulder_list_joint">
+            <joint name="${prefix}shoulder_lift_joint">
                 <command_interface name="position">
                     <param name="min">${-2*pi}</param>
